File: sharp_dsi_pcb/sharp_dsi.kicad_sch (KiCad schematic)
At the start: 1 part, among them U1 STM32F030F4Px

Commit message: pcb status gbr-v0.2
Parts:
- removed U1: STM32F030F4Px, Package_SO:TSSOP-20_4.4x6.5mm_P0.65mm, symbol MCU_ST_STM32F0:STM32F030F4Px
- added C1, C5: 10pF, Capacitor_SMD:C_0402_1005Metric, symbol Device:C
- added C10, C11, C12, C13, C14, C15, C16, C17, C18, C19, C2, C20, C21, C3, C4, C6, C7, C8, C9: 100nF, Capacitor_SMD:C_0402_1005Metric, symbol Device:C
- added D1, D2, D3, D4, D5, D6: LED, Resistor_SMD:R_0603_1608Metric, symbol Device:LED
- added J1: AYF333135, footprints:AYF333135, symbol jlywxy:AYF333135
- added J2: USB_C_Receptacle_USB2.0, Connector_USB:USB_C_Receptacle_HRO_TYPE-C-31-M-12, symbol Connector:USB_C_Receptacle_USB2.0
- added J3, J5: Conn_01x04_Male, Connector_PinHeader_2.54mm:PinHeader_1x04_P2.54mm_Vertical, symbol Connector:Conn_01x04_Male
- added J4: Conn_01x05, Connector_PinHeader_2.54mm:PinHeader_1x05_P2.54mm_Vertical, symbol Connector_Generic:Conn_01x05
- added J6: Conn_02x15_Counter_Clockwise, Connector_PinHeader_2.54mm:PinHeader_2x15_P2.54mm_Vertical, symbol Connector_Generic:Conn_02x15_Counter_Clockwise
- added R1, R2: 5.1k, Resistor_SMD:R_0603_1608Metric, symbol Device:R
- added R10, R5, R6, R7, R8, R9: 5.6k, Resistor_SMD:R_0603_1608Metric, symbol Device:R
- added R11, R12: 100k, Resistor_SMD:R_0603_1608Metric, symbol Device:R
- added R3: 220, Resistor_THT:R_Box_L8.4mm_W2.5mm_P5.08mm, symbol Device:R
- added R4: 10k, Resistor_SMD:R_0603_1608Metric, symbol Device:R
- added U1: XC6206PxxxMR, footprints:XC6206P502PR, symbol Regulator_Linear:XC6206PxxxMR
- added U2: SSD2828QN4, footprints:SSD2828QN4, symbol jlywxy:SSD2828QN4
- added U3: AMS1117, Package_TO_SOT_SMD:SOT-223-3_TabPin2, symbol Regulator_Linear:AMS1117
- added U4: XC6206PxxxMR, Package_TO_SOT_SMD:SOT-23, symbol Regulator_Linear:XC6206PxxxMR
- added U6: STM32F030F4Px, footprints:STM32F030F4P6, symbol MCU_ST_STM32F0:STM32F030F4Px
- added U7: ICL7660, Package_SO:SOIC-8_3.9x4.9mm_P1.27mm, symbol Regulator_SwitchedCapacitor:ICL7660
- added Y1: Crystal, Crystal:Crystal_SMD_5032-2Pin_5.0x3.2mm, symbol Device:Crystal
Connections:
- new net: J2.A5 (CC1), R1.1
- new net: D5.2 (A), R9.1
- new net: C10.1, U7.2 (CAP+)
- new net: C10.2, U7.4 (CAP-)
- new net: D4.2 (A), R8.1
- new net: D1.2 (A), R5.1
- new net: J4.3 (Pin_3), R3.2
- new net: D6.2 (A), R10.1
- new net: J2.B5 (CC2), R2.1
- new net: C5.1, U2.62 (TX_CLK_XIO), Y1.1
- new net: C1.1, U2.63 (TX_CLK_XIN), Y1.2
- new net: D2.2 (A), R6.1
- new net: D3.2 (A), R7.1
- new net: R4.2, U6.1 (BOOT0)
- new net 5v: C2.1, C4.1, C7.1, J2.A4 (VBUS), J2.A9 (VBUS), J2.B4 (VBUS), J2.B9 (VBUS), J3.1 (Pin_1), J3.2 (Pin_2), J4.1 (Pin_1), U1.3 (VI), U3.3 (VI), U4.3 (VI)
- new net GND: C1.2, C11.2, C12.1, C13.1, C14.2, C15.1, C16.2, C17.1, C18.2, C19.1, C2.2, C20.2, C21.1, C3.2, C4.2, C5.2, C6.2, C7.2, C8.2, C9.2, D1.1 (K), D2.1 (K), D3.1 (K), D4.1 (K), D5.1 (K), D6.1 (K), J1.16, J1.19, J1.22, J1.25, J1.28, J1.31, J1.6, J2.A1 (GND), J2.A12 (GND), J2.B1 (GND), J2.B12 (GND), J2.S1 (SHIELD), J3.4 (Pin_4), J4.2 (Pin_2), J5.3 (Pin_3), J6.19 (Pin_19), J6.20 (Pin_20), R1.2, R11.1, R12.1, R2.2, R4.1, U1.1 (GND), U2.12 (GND), U2.18 (PS1), U2.26 (SDC), U2.27 (SHUT), U2.3 (GND), U2.32 (GND), U2.6 (GND), U2.65 (GND), U2.67 (GND), U2.69 (GND), U2.9 (GND), U3.1 (ADJ), U4.1 (GND), U6.15 (VSS), U7.3 (GND)
- new net LCD_AVDD+: C8.1, C9.1, J1.10, U1.2 (VO), U7.8 (V+)
- new net LCD_AVDD-: C11.1, J1.11, U7.5 (VOUT)
- new net LCD_BL_19v: J1.1, J1.2, R3.1
- new net LCD_BL_GND: J1.3, J1.4, J4.4 (Pin_4)
- new net LCD_CTS0_ID0: J1.14, R12.2
- new net LCD_CTS1_ID1: J1.15, R11.2
- new net LCD_DSI_CLKN: J1.24, U2.8 (CLKN)
- new net LCD_DSI_CLKP: J1.23, U2.7 (CLKP)
- new net LCD_DSI_D0N: J1.27, U2.2 (DATAN0)
- new net LCD_DSI_D0P: J1.26, U2.1 (DATAP0)
- new net LCD_DSI_D1N: J1.21, U2.5 (DATAN1)
- new net LCD_DSI_D1P: J1.20, U2.4 (DATAP1)
- new net LCD_DSI_D2N: J1.18, U2.11 (DATAN2)
- new net LCD_DSI_D2P: J1.17, U2.10 (DATAP2)
- new net LCD_DSI_D3N: J1.30, U2.14 (DATAN3)
- new net LCD_DSI_D3P: J1.29, U2.13 (DATAP3)
- new net LCD_OUT_BLPWM: J1.12, R8.2
- new net LCD_OUT_HSYNC: J1.8, R10.2
- new net LCD_OUT_TE: J1.7, R9.2
- new net LCD_XRES: J1.13, U6.17 (PA9)
- new net SSD_CSX0: U2.59 (CSX0), U6.10 (PA4)
- new net SSD_MVDD: C15.2, C17.2, C19.2, C21.2, C3.1, U2.15 (MVDD), U2.31 (MVDD), U2.60 (MVDD), U2.66 (MVDD), U3.2 (VO)
- new net SSD_OUT_CLK: R7.2, U2.61 (SYS_CLK_OUT)
- new net SSD_PS0: C12.2, C13.2, C14.1, C16.1, C18.1, C20.1, C6.1, J1.9, J3.3 (Pin_3), J5.4 (Pin_4), R5.2, U2.16 (VDDIO), U2.17 (PS0), U2.33 (VDDIO), U2.64 (VDDIO), U2.68 (VDDIO), U4.2 (VO), U6.16 (VDD), U6.5 (VDDA)
- new net SSD_RESET: U2.22 (RESET), U6.9 (PA3)
- new net SSD_RGB_B0: J6.13 (Pin_13), U2.51 (DATA16)
- new net SSD_RGB_B1: J6.12 (Pin_12), U2.52 (DATA17)
- new net SSD_RGB_B2: J6.10 (Pin_10), U2.53 (DATA18)
- new net SSD_RGB_B3: J6.9 (Pin_9), U2.54 (DATA19)
- new net SSD_RGB_B4: J6.8 (Pin_8), U2.55 (DATA20)
- new net SSD_RGB_B5: J6.7 (Pin_7), U2.56 (DATA21)
- new net SSD_RGB_B6: J6.6 (Pin_6), U2.57 (DATA22)
- new net SSD_RGB_B7: J6.5 (Pin_5), U2.58 (DATA23)
- new net SSD_RGB_DEN: J6.3 (Pin_3), U2.28 (DEN)
- new net SSD_RGB_G0: J6.22 (Pin_22), U2.43 (DATA8)
- new net SSD_RGB_G1: J6.21 (Pin_21), U2.44 (DATA9)
- new net SSD_RGB_G2: J6.11 (Pin_11), U2.45 (DATA10)
- new net SSD_RGB_G3: J6.18 (Pin_18), U2.46 (DATA11)
- new net SSD_RGB_G4: J6.17 (Pin_17), U2.47 (DATA12)
- new net SSD_RGB_G5: J6.16 (Pin_16), U2.48 (DATA13)
- new net SSD_RGB_G6: J6.15 (Pin_15), U2.49 (DATA14)
- new net SSD_RGB_G7: J6.14 (Pin_14), U2.50 (DATA15)
- new net SSD_RGB_HSYNC: J6.1 (Pin_1), U2.29 (HSYNC)
- new net SSD_RGB_PCLK: J6.4 (Pin_4), U2.30 (PCLK)
- new net SSD_RGB_R0: J6.30 (Pin_30), U2.35 (DATA0)
- new net SSD_RGB_R1: J6.29 (Pin_29), U2.36 (DATA1)
- new net SSD_RGB_R2: J6.28 (Pin_28), U2.37 (DATA2)
- new net SSD_RGB_R3: J6.27 (Pin_27), U2.38 (DATA3)
- new net SSD_RGB_R4: J6.26 (Pin_26), U2.39 (DATA4)
- new net SSD_RGB_R5: J6.25 (Pin_25), U2.40 (DATA5)
- new net SSD_RGB_R6: J6.24 (Pin_24), U2.41 (DATA6)
- new net SSD_RGB_R7: J6.23 (Pin_23), U2.42 (DATA7)
- new net SSD_RGB_VSYNC: J6.2 (Pin_2), U2.34 (VSYNC)
- new net SSD_SCK: U2.25 (SCK), U6.11 (PA5)
- new net SSD_SDI: U2.24 (SDI), U6.13 (PA7)
- new net SSD_SDO: U2.23 (SDO), U6.12 (PA6)
- new net ST_PB1: R6.2, U6.14 (PB1)
- new net ST_SWCLK: J5.1 (Pin_1), U6.20 (PA14)
- new net ST_SWDIO: J5.2 (Pin_2), U6.19 (PA13)
- no-connect marks 0 -> 17
Other:
- note added: "LCD_AVDD_5v_SOT89"
- note added: "REVERSED CONNECTOR BOTTOM CONTACT"
- note added: "SSD_LCD_ST_VDDIO_3v3_SOT23"
- note added: "SSD_MVDD_1.2_SOT223"
- company: (none) -> github/jlywxy | the Monazite workshop
- title: (none) -> Sharp DSI Eva
